File: ELM327_V1/ELM327/_autosave-ELM327.sch (KiCad schematic (older format))
At the start: 7 parts

Commit message: Update enable git
Parts:
- gave numbers to parts that had none: 7
Changed lines of the file:
@@
 $EndSheet
 $Comp
-L power:+3.3V #PWR?
+L power:+3.3V #PWR0101
 U 1 1 61B8CF39
 P 4450 1450
-F 0 "#PWR?" H 4450 1300 50  0001 C CNN
+F 0 "#PWR0101" H 4450 1300 50  0001 C CNN
 F 1 "+3.3V" H 4465 1623 50  0000 C CNN
 F 2 "" H 4450 1450 50  0001 C CNN
@@
 $EndComp
 $Comp
-L power:+3.3V #PWR?
+L power:+3.3V #PWR0102
 U 1 1 61B8DD97
 P 5975 1375
-F 0 "#PWR?" H 5975 1225 50  0001 C CNN
+F 0 "#PWR0102" H 5975 1225 50  0001 C CNN
 F 1 "+3.3V" H 5990 1548 50  0000 C CNN
 F 2 "" H 5975 1375 50  0001 C CNN
@@
 	5975 2050 6450 2050
 $Comp
-L power:GND #PWR?
+L power:GND #PWR0103
 U 1 1 61B8F0DF
 P 6450 4900
-F 0 "#PWR?" H 6450 4650 50  0001 C CNN
+F 0 "#PWR0103" H 6450 4650 50  0001 C CNN
 F 1 "GND" H 6455 4727 50  0000 C CNN
 F 2 "" H 6450 4900 50  0001 C CNN
@@
 	6450 4900 6450 4850
 $Comp
-L Device:C C?
+L Device:C C3
 U 1 1 61B9108D
 P 5525 1875
-F 0 "C?" V 5777 1875 50  0000 C CNN
+F 0 "C3" V 5777 1875 50  0000 C CNN
 F 1 "0.1uF" V 5686 1875 50  0000 C CNN
 F 2 "" H 5563 1725 50  0001 C CNN
@@
 $EndComp
 $Comp
-L Device:C C?
+L Device:C C2
 U 1 1 61B91E1D
 P 5525 1475
-F 0 "C?" V 5777 1475 50  0000 C CNN
+F 0 "C2" V 5777 1475 50  0000 C CNN
 F 1 "0.1uF" V 5686 1475 50  0000 C CNN
 F 2 "" H 5563 1325 50  0001 C CNN
@@
 	5000 1475 5375 1475
 $Comp
-L power:GND #PWR?
+L power:GND #PWR0104
 U 1 1 61B9CE7F
 P 4775 1700
-F 0 "#PWR?" H 4775 1450 50  0001 C CNN
+F 0 "#PWR0104" H 4775 1450 50  0001 C CNN
 F 1 "GND" H 4780 1527 50  0000 C CNN
 F 2 "" H 4775 1700 50  0001 C CNN
@@
 	5000 1675 5000 1475
 $Comp
-L Device:R R?
+L Device:R R1
 U 1 1 61BA0A50
 P 4450 1675
-F 0 "R?" H 4520 1721 50  0000 L CNN
+F 0 "R1" H 4520 1721 50  0000 L CNN
 F 1 "10K" H 4520 1630 50  0000 L CNN
 F 2 "" V 4380 1675 50  0001 C CNN
@@
 	4450 2250 5850 2250
 $Comp
-L Device:C C?
+L Device:C C1
 U 1 1 61BA1834
 P 4125 2250
-F 0 "C?" V 4377 2250 50  0000 C CNN
+F 0 "C1" V 4377 2250 50  0000 C CNN
 F 1 "1uF" V 4286 2250 50  0000 C CNN
 F 2 "" H 4163 2100 50  0001 C CNN
@@
 Connection ~ 4450 2250
 $Comp
-L power:GND #PWR?
+L power:GND #PWR0105
 U 1 1 61BA1F72
 P 3800 2300
-F 0 "#PWR?" H 3800 2050 50  0001 C CNN
+F 0 "#PWR0105" H 3800 2050 50  0001 C CNN
 F 1 "GND" H 3805 2127 50  0000 C CNN
 F 2 "" H 3800 2300 50  0001 C CNN
@@
 $EndSheet
 $Comp
-L Connector_Generic:Conn_02x02_Counter_Clockwise J?
+L Connector_Generic:Conn_02x02_Counter_Clockwise J2
 U 1 1 61C3853B
 P 9650 1375
-F 0 "J?" H 9700 1592 50  0000 C CNN
+F 0 "J2" H 9700 1592 50  0000 C CNN
 F 1 "Conn_02x02_Counter_Clockwise" H 9700 1501 50  0000 C CNN
 F 2 "" H 9650 1375 50  0001 C CNN
@@
 PROGRAM_PORT_RX
 $Comp
-L Connector_Generic:Conn_02x02_Counter_Clockwise J?
+L Connector_Generic:Conn_02x02_Counter_Clockwise J1
 U 1 1 61C5AFB5
 P 9525 3250
-F 0 "J?" H 9575 3467 50  0000 C CNN
+F 0 "J1" H 9575 3467 50  0000 C CNN
 F 1 "Conn_02x02_Counter_Clockwise" H 9575 3376 50  0000 C CNN
 F 2 "" H 9525 3250 50  0001 C CNN
@@
 ESP_TO_ELM_RX_IN
 $Comp
-L RF_Module:ESP32-WROOM-32 U?
+L RF_Module:ESP32-WROOM-32 U1
 U 1 1 61C67283
 P 6450 3450
-F 0 "U?" H 6450 5031 50  0000 C CNN
+F 0 "U1" H 6450 5031 50  0000 C CNN
 F 1 "ESP32-WROOM-32" H 6450 4940 50  0000 C CNN
 F 2 "RF_Module:ESP32-WROOM-32" H 6450 1950 50  0001 C CNN
